File: 2605268-Juan Cruz-Microduino/2605268-Juan Cruz-Microduino.kicad_pcb (KiCad board)
At the start: 2 copper layers, 14 parts, among them J1 USB_A_UCC, J2 Conn_01x10_Socket, U1 ATtiny85-20S

Commit message: Add files via upload
Parts:
- C1: value C -> 0.1 u
- D1: footprint Diode_SMD:D_MELF_Handsoldering -> Diode_SMD:D_MiniMELF
- D2: value D_Zener -> 3.6V 1/2mW
- D3: value LED -> 3.6V 1/2mW; footprint Library:LED.R -> Diode_SMD:D_SOD-123
- D4: value LED -> LED Green; footprint Library:LED.R -> Library_UCC:led_UCC
- D5: value D_Zener -> LED; footprint Diode_SMD:D_SOD-123 -> Library_UCC:led_UCC
- J1: value USB_A_UCC -> USB_A; footprint Library:USB_A_UCC -> Library_UCC:USB_A_UCC
- J2: value Conn_01x10_Socket -> Header
- R1: value R -> 1.5KΩ 5% 1/8W
- R2, R3: value R -> 68Ω 5% 1/8W
- R4: value R -> 330Ω 5% 1/8W; footprint Capacitor_SMD:C_0805_2012Metric_Pad1.18x1.45mm_HandSolder -> Resistor_SMD:R_0805_2012Metric_Pad1.20x1.40mm_HandSolder
- R5: value R -> 330Ω 5% 1/8W
- U1: value ATtiny85-20S -> ATtiny13-20SU
- moved D3 60.4 mm to (140.3, 87.6), turned to 0 degrees
- moved R4 53.0 mm to (126.9, 92.1)
- moved C1 52.2 mm to (124.0, 87.6), turned to 180 degrees
- moved J2 51.8 mm to (119.9, 99.1)
- moved D4 51.8 mm to (131.4, 93.7)
- moved U1 51.2 mm to (140.3, 93.0)
- moved D2 51.2 mm to (123.4, 84.6), turned to 180 degrees
- moved R1 51.1 mm to (128.9, 86.1), turned to 90 degrees
- moved R2 51.1 mm to (132.9, 86.1), turned to 90 degrees
- moved D1 51.0 mm to (118.9, 90.6)
- moved R3 50.6 mm to (140.4, 84.6)
- moved R5 50.4 mm to (125.9, 95.6), turned to 180 degrees
- moved D5 47.4 mm to (122.3, 93.1), turned to -90 degrees
- moved J1 46.8 mm to (122.4, 78.3)
Connections:
- D3 pad 2: Net-(D3-A) -> GND
- D4 pad 2: +5V -> Net-(D4-A)
- D5 pad 2: GND -> +5V
- J1 pad 3: Net-(D5-K) -> Net-(D3-K)
- J2 pad 5: Net-(D3-A) -> Net-(D4-A)
- R2 pad 1: Net-(D5-K) -> Net-(J2-Pin_7)
- R2 pad 2: Net-(J2-Pin_8) -> Net-(D2-K)
- R3 pad 1: Net-(D2-K) -> Net-(J2-Pin_8)
- R3 pad 2: Net-(J2-Pin_7) -> Net-(D3-K)
- R4 pad 1: Net-(D3-K) -> GND
- R4 pad 2: GND -> Net-(D4-K)
- R5 pad 1: Net-(D4-K) -> GND
- R5 pad 2: GND -> Net-(D5-K)
- U1 pad 6: Net-(D3-A) -> Net-(D4-A)
Routing:
- net GND: track 30.8 -> 57.3 mm
- net Net-(D3-K): track 0.00 -> 23.3 mm
- net +5V: track 19.4 -> 34.7 mm
- net Net-(D4-A): track 0.00 -> 11.0 mm
- net Net-(D3-A): track 8.90 -> 0.00 mm
- net Net-(J2-Pin_7): track 10.5 -> 17.3 mm
- net Net-(D5-K): track 0.00 -> 5.86 mm
- net Net-(J2-Pin_9): track 4.86 -> 0.00 mm
- net Net-(D1-A): track 14.9 -> 10.8 mm
- net Net-(D4-K): track 0.00 -> 4.04 mm
- net Net-(J2-Pin_4): track 12.0 -> 13.8 mm
- net Net-(J2-Pin_8): track 11.5 -> 10.4 mm
- net Net-(J2-Pin_6): track 6.59 -> 7.68 mm
- net Net-(D2-K): track 19.5 -> 18.6 mm
- added copper zone on F.Cu, net (none)
Other:
- board outline added: 31 x 29 mm
